File: Hardware/modules/ACIA2/ACIA2.kicad_sch (KiCad schematic)
At the start: 43 parts, among them J10 COM2/4, J11 PORT2, J12 Bus_PCI_6502, J8 COM1/3, J9 PORT1, U10 MAX232, U11 6551, U12 MAX232, U13 MAX232, U14 6551, U15 74HC138, U16 74HC138, U9 MAX232, X2 1.8432MHz

Commit message: Add review comments and make new branch
Other:
- note added: "Stützkondensatoren an MAX Chips min 1µF besser 10µF"
Changed lines of the file:
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@@
+		)
+	)
+	(text "Stützkondensatoren an MAX Chips min 1µF besser 10µF"
+		(exclude_from_sim no)
+		(at 163.195 367.03 0)
+		(effects
+			(font
+				(size 2.54 2.54)
+				(thickness 0.508)
+				(bold yes)
+			)
 		)
 	)
