File: Hardware/modules/Bank_IRQ/Bank_IRQ.kicad_sch (KiCad schematic)
At the start: 27 parts, among them J2 Bus_PCI_6502, U1 74HC00, U2 74HC138, U3 6525

Commit message: Add review comments and make new branch
Other:
- note added: "Decoding anschauen?"
Changed lines of the file:
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@@
+		)
+	)
+	(text "Decoding anschauen?"
+		(exclude_from_sim no)
+		(at 149.225 49.53 0)
+		(effects
+			(font
+				(size 2.54 2.54)
+				(thickness 0.508)
+				(bold yes)
+			)
 		)
 	)
