File: Hardware/modules/Bus_Card/Bus_Card.kicad_sch (KiCad schematic)
At the start: 19 parts, among them J1 DC In, SW1 RESET, SW2 NMI, U1 SY317, U2 SY317

Commit message: Add review comments and make new branch
Other:
- note added: "Stützkondensatoren den LDOs 10µF"
Changed lines of the file:
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@@
+		)
+	)
+	(text "Stützkondensatoren den LDOs 10µF"
+		(exclude_from_sim no)
+		(at 351.155 217.17 0)
+		(effects
+			(font
+				(size 2.54 2.54)
+				(thickness 0.508)
+				(bold yes)
+			)
 		)
 	)
