File: Hardware/modules/CPU/CPU.kicad_sch (KiCad schematic)
At the start: 16 parts, among them J1 ABORT, J2 SO/MX, J3 Bus_PCI_6502, J5 Bank Bridge A, J6 Bank Bridge B, J7 Bank Bridge C, U1 65C02 / 65816, U2 74HC00, U3 74HC245, U4 74LS573

Commit message: Add review comments and make new branch
Other:
- note added: "100nF an RESET"
Changed lines of the file:
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@@
+		)
+	)
+	(text "100nF an RESET"
+		(exclude_from_sim no)
+		(at 153.67 22.225 0)
+		(effects
+			(font
+				(size 2.54 2.54)
+				(thickness 0.508)
+				(bold yes)
+			)
 		)
 	)
