File: Hardware/modules/LCD_IRQ/LCD_IRQ.kicad_sch (KiCad schematic)
At the start: 18 parts, among them J1 Bus_PCI_6502, U1 74HC138, U2 W65C22SxP

Commit message: Add review comments and make new branch
Other:
- note added: "Stützkondensatoren an LCD min 1µF besser 10µF"
Changed lines of the file:
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@@
+		)
+	)
+	(text "Stützkondensatoren an LCD min 1µF besser 10µF"
+		(exclude_from_sim no)
+		(at 153.67 114.3 0)
+		(effects
+			(font
+				(size 2.54 2.54)
+				(thickness 0.508)
+				(bold yes)
+			)
 		)
 	)
