File: Hardware/modules/PIA_LED/PIA_LED.kicad_sch (KiCad schematic)
At the start: 39 parts, among them J1 Bus_PCI_6502, J2 PIA_A, J3 PIA_B, U1 6520, U2 74HC138

Commit message: Add review comments and make new branch
Other:
- note added: "Decoding anschauen?? Port 16 vs Port 28"
Changed lines of the file:
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@@
+		)
+	)
+	(text "Decoding anschauen??\nPort 16 vs Port 28"
+		(exclude_from_sim no)
+		(at 143.51 71.755 0)
+		(effects
+			(font
+				(size 2.54 2.54)
+				(thickness 0.508)
+				(bold yes)
+			)
 		)
 	)
