File: Hardware/modules/SID/SID.kicad_sch (KiCad schematic)
At the start: 14 parts, among them J1 Bus_PCI_6502, J2 POT_X, J3 POT_Y, J4 POT_X, U1 74HC138, U2 8580

Commit message: Add review comments and make new branch
Other:
- note added: "Stützkondensatoren am Audio Chip min 1µF besser 10µF"
Changed lines of the file:
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@@
+		)
+	)
+	(text "Stützkondensatoren am Audio Chip min 1µF besser 10µF"
+		(exclude_from_sim no)
+		(at 162.56 161.29 0)
+		(effects
+			(font
+				(size 2.54 2.54)
+				(thickness 0.508)
+				(bold yes)
+			)
 		)
 	)
